File: Hardware/Rele wifi/Rele wifi.kicad_sch (KiCad schematic)
At the start: 8 parts, among them Q1 BF457, U1 ESP8266

Commit message: actu
Parts:
- removed U1: ESP8266, symbol ESP32-DEVKITC-32xd:ESP8266
- added U2: ~, symbol ESP32-DEVKITC-32xd:ESP8266
Connections:
- net at BZ1.1 (+): now also U2. (3.3V)
- net at BZ1.2 (-): now also U2. (3.3V)
Other:
- moved on the sheet: BZ1, C1, C2, D1, D2, Q1, R1
