File: Hardware/Rele wifi/Rele wifi.kicad_sch (KiCad schematic)
At the start: 16 parts, among them K1 G5LE-1, Q1 BF457, Q2 BF457, SW1 SW_Push, U1 PC817

Commit message: actu
Parts:
- removed U2: ~, symbol ESP32-DEVKITC-32xd:ESP8266
- added J1, J2: Screw_Terminal_01x02, TerminalBlock:TerminalBlock_MaiXu_MX126-5.0-02P_1x02_P5.00mm, symbol Connector:Screw_Terminal_01x02
- added J3, J4: Conn_01x15_Pin, Connector_PinHeader_1.00mm:PinHeader_1x15_P1.00mm_Vertical, symbol Connector:Conn_01x15_Pin
- BZ1: footprint (none) -> Buzzer_Beeper:Buzzer_12x9.5RM7.6
- C1: footprint (none) -> Capacitor_SMD:C_0201_0603Metric
- C2: footprint (none) -> Capacitor_THT:CP_Radial_D5.0mm_P2.50mm
- D1: footprint (none) -> LED_THT:LED_D3.0mm
- R1, R3, R4: footprint (none) -> Resistor_SMD:R_0201_0603Metric
- R2: value 220K -> 220; footprint (none) -> Resistor_SMD:R_0201_0603Metric
- R5: value 220k -> 220; footprint (none) -> Resistor_SMD:R_0201_0603Metric
- SW1: footprint (none) -> Button_Switch_THT:SW_PUSH_6mm_H5mm
Connections:
- net GND: now also J2.2 (Pin_2), J4.14 (Pin_14); no longer K1.5
- net VCC: now also J2.1 (Pin_1), J4.15 (Pin_15)
- net at R4.1, SW1.1: now also J3.9 (Pin_9)
- net at R2.1: now also J3.7 (Pin_7)
- net at R4.2: now also J3.15 (Pin_15)
- net at U1.2: now also D1.2 (A)
- net at U1.4: now also D2.1 (K), K1.5, J3.6 (Pin_6); no longer K1.3
- net at D2.2 (A): now also K1.2, Q2.2 (C)
- net at BZ1.1 (+): now also K1.3; no longer K1.1
- net at BZ1.2 (-): now also K1.1; no longer K1.2
- net at D1.1 (K): now also J3.8 (Pin_8)
- net at K1.4: no longer Q2.2 (C)
Other:
- moved on the sheet: BZ1, C1, C2, D1, D2, K1, Q1, R1, R2, R3, R4, R5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

Commit message: placa
Parts:
- removed BZ1: Buzzer, Buzzer_Beeper:Buzzer_12x9.5RM7.6, symbol Device:Buzzer
- removed C1: C, Capacitor_SMD:C_0201_0603Metric, symbol Device:C
- removed C2: C_Polarized, Capacitor_THT:CP_Radial_D5.0mm_P2.50mm, symbol Device:C_Polarized
- removed D2: 1N4007, Diode_THT:D_DO-41_SOD81_P10.16mm_Horizontal, symbol Diode:1N4007
- removed J3, J4: Conn_01x15_Pin, Connector_PinHeader_1.00mm:PinHeader_1x15_P1.00mm_Vertical, symbol Connector:Conn_01x15_Pin
- removed Q1, Q2: BF457, Package_TO_SOT_THT:TO-126-3_Vertical, symbol Transistor_BJT:BF457
- removed R4: 10K, Resistor_SMD:R_0201_0603Metric, symbol Device:R
- removed R5: 220, Resistor_SMD:R_0201_0603Metric, symbol Device:R
- removed SW1: SW_Push, Button_Switch_THT:SW_PUSH_6mm_H5mm, symbol Switch:SW_Push
- removed U1: PC817, Package_DIP:DIP-4_W7.62mm, symbol Isolator:PC817
- added D3: 1N4007, Diode_SMD:D_0805_2012Metric, symbol local_lib:1N4007
- added Q1: BC414, Package_TO_SOT_THT:TO-92_Inline, symbol Transistor_BJT:BC414
- added U1: ESP8266-DEVKITC-02U-F, esp32:ESP8266NA, symbol ESP8266-DEVKITC-02U-F:ESP8266-DEVKITC-02U-F
- added U5: PC817, Package_DIP:DIP-4_W7.62mm, symbol local_lib:PC817
- D1: footprint LED_THT:LED_D3.0mm -> LED_THT:LED_D3.0mm_Clear
- R1: value R -> 220; footprint Resistor_SMD:R_0201_0603Metric -> Resistor_SMD:R_0805_2012Metric
- R2: value 220 -> 1K; footprint Resistor_SMD:R_0201_0603Metric -> Resistor_SMD:R_0805_2012Metric
- R3: value 10K -> 1K; footprint Resistor_SMD:R_0201_0603Metric -> Resistor_SMD:R_0805_2012Metric
Connections:
- net VCC is gone; now on an unnamed net: J2.1 (Pin_1)
- net GND: now also J1.2 (Pin_2), Q1.3 (E), U1.J2_14 (GND_J2_14), U5.2; no longer J2.2 (Pin_2)
- net +5V: now reaches K1.5
- net +5V: now also J1.1 (Pin_1), R1.2, D3.1 (K), U1.J2_15 (GND_J2_15), U5.4
- net at K1.2: now also D1.1 (K), D3.2 (A), Q1.1 (C)
- net at R2.1: now also U5.3
- net at R2.2: now also Q1.2 (B)
- net at K1.1: now also J2.2 (Pin_2)
- net at D1.2 (A): now also R1.1
- net GPIO6: now reaches R3.1
- net GPIO6: now also U1.J2_9 (IO15)
- net at R3.2: now also U5.1
Other:
- moved on the sheet: K1

Commit message: pcb
Parts:
- removed J2: Screw_Terminal_01x02, TerminalBlock:TerminalBlock_MaiXu_MX126-5.0-02P_1x02_P5.00mm, symbol Connector:Screw_Terminal_01x02
- removed Q1: BC414, Package_TO_SOT_THT:TO-92_Inline, symbol Transistor_BJT:BC414
- added J2: Screw_Terminal_01x03, TerminalBlock:TerminalBlock_MaiXu_MX126-5.0-03P_1x03_P5.00mm, symbol Connector:Screw_Terminal_01x03
- added Q2: BC337, Package_TO_SOT_THT:TO-92_Inline, symbol Transistor_BJT:BC337
Connections:
- net GND: now also Q2.3 (E)
- net NC: now reaches K1.3
- net NC: now also J2.2 (Pin_2)
- net COM: now reaches K1.1
- net COM: now also J2.3 (Pin_3)
- net at D1.1 (K), D3.2 (A), K1.2: now also Q2.1 (C)
- net at R2.2: now also Q2.2 (B)
- net NO: now reaches K1.4
- net NO: now also J2.1 (Pin_1)

Commit message: actu
Parts:
- added J3: Screw_Terminal_01x02, TerminalBlock:TerminalBlock_MaiXu_MX126-5.0-02P_1x02_P5.00mm, symbol Connector:Screw_Terminal_01x02
- U5: footprint Package_DIP:DIP-4_W7.62mm -> Package_SO:SOP-4_4.4x2.6mm_P1.27mm
Changed lines of the file:
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@@
+	)
+	(symbol
+		(lib_id "Connector:Screw_Terminal_01x02")
+		(at 240.03 59.69 0)
+		(unit 1)
+		(exclude_from_sim no)
+		(in_bom yes)
+		(on_board yes)
+		(dnp no)
+		(fields_autoplaced yes)
+		(property "Reference" "J3"
+			(at 242.57 60.9599 0)
+			(effects
+				(font
+					(size 1.27 1.27)
+				)
+				(justify left)
+			)
+		)
+		(property "Value" "Screw_Terminal_01x02"
+			(at 242.57 62.2299 0)
+			(effects
+				(font
+					(size 1.27 1.27)
+				)
+				(justify left)
+				(hide yes)
+			)
+		)
+		(property "Footprint" "TerminalBlock:TerminalBlock_MaiXu_MX126-5.0-02P_1x02_P5.00mm"
+			(at 240.03 59.69 0)
+			(effects
+				(font
+					(size 1.27 1.27)
+				)
+				(hide yes)
+			)
+		)
+		(property "Datasheet" "~"
+			(at 240.03 59.69 0)
+			(effects
+				(font
+					(size 1.27 1.27)
+				)
+				(hide yes)
+			)
+		)
+		(property "Description" "Generic screw terminal, single row, 01x02, script generated (kicad-library-utils/schlib/autogen/connector/)"
+			(at 240.03 59.69 0)
+			(effects
+				(font
+					(size 1.27 1.27)
+				)
+				(hide yes)
+			)
+		)
+		(pin "1"
+		)
+		(pin "2"
+		)
+		(instances
+			(project "Rele wifi"
+				(path "/ffdbb2c2-c0c7-4e42-be77-90fd93012b1e"
+					(reference "J3")
+					(unit 1)
+				)
+			)
+		)
 	)
 	(symbol
@@
 			)
 		)
-		(property "Footprint" "Package_DIP:DIP-4_W7.62mm"
+		(property "Footprint" "Package_SO:SOP-4_4.4x2.6mm_P1.27mm"
 			(at 149.86 72.39 0)
 			(effects

Commit message: actu
Parts:
- removed U1: ESP8266-DEVKITC-02U-F, esp32:ESP8266NA, symbol ESP8266-DEVKITC-02U-F:ESP8266-DEVKITC-02U-F
- added U2: ~, ESP32_Footprints:ESP32_30pin, symbol esp32_30pin_revised:ESP32_30Pin
Connections:
- net +5V: now also U2.1 (VIN)
- net GND: now also U2.2 (GND)
- net GPIO6: now also U2.7 (GPIO26)
Other:
- moved on the sheet: D1, D3, J1, J2, J3, K1, Q2, R1, R2, R3, U5

Commit message: actu pcb
Parts:
- removed J3: Screw_Terminal_01x02, TerminalBlock:TerminalBlock_MaiXu_MX126-5.0-02P_1x02_P5.00mm, symbol Connector:Screw_Terminal_01x02
- added D2: LED IR, LED_THT:LED_D3.0mm_Clear, symbol Device:LED
- added Q1: BC337, Package_TO_SOT_THT:TO-92_Inline, symbol Transistor_BJT:BC337
- added R4: 220, Resistor_SMD:R_0805_2012Metric, symbol Device:R
- added R5: 47, Resistor_SMD:R_0805_2012Metric, symbol Device:R
Connections:
- net +5V: now also R5.1
- net GND: now also Q1.3 (E)
- net GPIO7: now reaches U2.8 (GPIO25)
- net GPIO7: now also R4.2
- new net: D2.2 (A), R5.2
- new net: D2.1 (K), Q1.1 (C)
- new net: Q1.2 (B), R4.1
