File: Hardware/Rele wifi/Rele wifi.kicad_pcb (KiCad board)
At the start: 2 copper layers, 19 parts, among them J1 Screw_Terminal_01x02, J2 Screw_Terminal_01x02, J3 Conn_01x15_Pin, J4 Conn_01x15_Pin, K1 G5LE-1, Q1 BF457, Q2 BF457, SW1 SW_Push, U1 PC817

Commit message: placa
Parts:
- removed BZ1: Buzzer, Buzzer_Beeper:Buzzer_12x9.5RM7.6
- removed C1: C, Capacitor_SMD:C_0201_0603Metric
- removed C2: C_Polarized, Capacitor_THT:CP_Radial_D5.0mm_P2.50mm
- removed D2: 1N4007, Diode_THT:D_DO-41_SOD81_P10.16mm_Horizontal
- removed J3, J4: Conn_01x15_Pin, Connector_PinHeader_1.00mm:PinHeader_1x15_P1.00mm_Vertical
- removed Q2: BF457, Package_TO_SOT_THT:TO-126-3_Vertical
- removed R4: 10K, Resistor_SMD:R_0201_0603Metric
- removed R5: 220, Resistor_SMD:R_0201_0603Metric
- removed SW1: SW_Push, Button_Switch_THT:SW_PUSH_6mm_H5mm
- added D3: 1N4007, Diode_SMD:D_0805_2012Metric, B.Cu at (193.8, 69.7)
- added U5: PC817, Package_DIP:DIP-4_W7.62mm, F.Cu at (195.4, 63.0)
- D1: footprint LED_THT:LED_D3.0mm -> LED_THT:LED_D3.0mm_Clear
- Q1: value BF457 -> BC414; footprint Package_TO_SOT_THT:TO-126-3_Vertical -> Package_TO_SOT_THT:TO-92_Inline
- R1: value R -> 220; footprint Resistor_SMD:R_0201_0603Metric -> Resistor_SMD:R_0805_2012Metric; moved to B.Cu
- R2: value 220 -> 1K; footprint Resistor_SMD:R_0201_0603Metric -> Resistor_SMD:R_0805_2012Metric; moved to B.Cu
- R3: value 10K -> 1K; footprint Resistor_SMD:R_0201_0603Metric -> Resistor_SMD:R_0805_2012Metric; moved to B.Cu
- U1: value PC817 -> ESP8266-DEVKITC-02U-F; footprint Package_DIP:DIP-4_W7.62mm -> esp32:ESP8266NA
- moved R2 115.5 mm to (208.1, 61.0)
- moved R3 110.5 mm to (190.7, 63.0)
- moved R1 92.8 mm to (192.9, 78.7), turned to 90 degrees
- moved Q1 85.5 mm to (214.2, 62.2), turned to 90 degrees
- moved D1 59.3 mm to (190.9, 87.2), turned to 90 degrees
- moved K1 49.5 mm to (216.2, 76.1), turned to -90 degrees
- moved U1 38.2 mm to (168.4, 77.0), turned to 180 degrees
- moved J1 37.5 mm to (211.6, 93.0)
- moved J2 35.4 mm to (197.0, 93.0)
Connections:
- J1 pad 1: unconnected-(J1-Pin_1-Pad1) -> +5V
- J1 pad 2: unconnected-(J1-Pin_2-Pad2) -> GND
- J2 pad 1: VCC -> Net-(J2-Pin_1)
- J2 pad 2: GND -> Net-(J2-Pin_2)
- K1 pad 1: Net-(BZ1--) -> Net-(J2-Pin_2)
- K1 pad 2: Net-(D2-A) -> Net-(D1-K)
- K1 pad 3: Net-(BZ1-+) -> Net-(J2-Pin_1)
- K1 pad 5: Net-(D2-K) -> +5V
- Q1 pad 1: unconnected-(Q1-E-Pad1) -> Net-(D1-K)
- Q1 pad 2: unconnected-(Q1-C-Pad2) -> Net-(Q1-B)
- Q1 pad 3: unconnected-(Q1-B-Pad3) -> GND
- R1 pad 1: unconnected-(R1-Pad1) -> Net-(D1-A)
- R1 pad 2: unconnected-(R1-Pad2) -> +5V
- R2 pad 2: Net-(R2-Pad2) -> Net-(Q1-B)
- R3 pad 1: Net-(R3-Pad1) -> GPIO6
Routing:
- net +5V: track 0.00 -> 138.7 mm
- net Net-(D1-K): track 0.00 -> 27.7 mm
- net Net-(J2-Pin_1): track 0.00 -> 24.9 mm
- net Net-(J2-Pin_2): track 0.00 -> 24.3 mm
- net GPIO6: track 0.00 -> 17.5 mm
- net Net-(R2-Pad1): track 0.00 -> 8.12 mm
- net Net-(D1-A): track 0.00 -> 5.85 mm
- net Net-(Q1-B): track 0.00 -> 5.21 mm
- net Net-(R3-Pad2): track 0.00 -> 3.88 mm
- added copper zone on B.Cu, net GND
Other:
- board outline added: 70 x 45 mm

Commit message: pcb
Parts:
- removed Q1: BC414, Package_TO_SOT_THT:TO-92_Inline
- added Q2: BC337, Package_TO_SOT_THT:TO-92_Inline, F.Cu at (214.2, 62.2)
- J2: value Screw_Terminal_01x02 -> Screw_Terminal_01x03; footprint TerminalBlock:TerminalBlock_MaiXu_MX126-5.0-02P_1x02_P5.00mm -> TerminalBlock:TerminalBlock_MaiXu_MX126-5.0-03P_1x03_P5.00mm
- moved D1 6.06 mm to (187.5, 82.2)
- moved J2 5.05 mm to (191.9, 93.0)
- moved U5 3.30 mm to (195.4, 59.7)
- moved R3 2.48 mm to (190.1, 60.6), turned to 90 degrees
- moved R2 1.45 mm to (207.4, 62.2)
Connections:
- K1 pad 1: Net-(J2-Pin_2) -> Net-(J2-Pin_3)
- K1 pad 3: Net-(J2-Pin_1) -> Net-(J2-Pin_2)
- K1 pad 4: unconnected-(K1-Pad4) -> Net-(J2-Pin_1)
Routing:
- net Net-(J2-Pin_3): track 0.00 -> 26.1 mm
- net Net-(D1-K): track 27.7 -> 48.0 mm
- net +5V: track 138.7 -> 120.3 mm
- net Net-(J2-Pin_1): track 24.9 -> 17.3 mm
- net Net-(J2-Pin_2): track 24.3 -> 29.9 mm
- net Net-(R2-Pad1): track 8.12 -> 3.48 mm
- net GPIO6: track 17.5 -> 19.1 mm
- net Net-(R3-Pad2): track 3.88 -> 5.32 mm
- net Net-(Q2-B): track 5.21 -> 6.46 mm

Commit message: actu
Parts:
- added J3: Screw_Terminal_01x02, TerminalBlock:TerminalBlock_MaiXu_MX126-5.0-02P_1x02_P5.00mm, F.Cu at (185.3, 93.0)
- U5: footprint Package_DIP:DIP-4_W7.62mm -> Package_SO:SOP-4_4.4x2.6mm_P1.27mm; moved to B.Cu
- moved J2 5.54 mm to (197.5, 93.0)
- moved U5 3.88 mm to (198.8, 61.5)
- moved J1 3.21 mm to (214.8, 93.0)
- moved R3 3.01 mm to (187.4, 62.1), turned to 0 degrees
- moved R2 1.52 mm to (206.8, 60.8)
- moved U1 0.60 mm to (167.8, 76.9)
- moved Q2 0.10 mm to (214.2, 62.1)
Connections:
- net Net-(J2-Pin_1) renamed NO
- net Net-(J2-Pin_2) renamed NC
- net Net-(J2-Pin_3) renamed COM
Routing:
- net +5V: track 120.3 -> 126.4 mm
- net NC: track 29.9 -> 25.1 mm
- net COM: track 26.1 -> 22.1 mm
- net NO: track 17.3 -> 14.1 mm
- net GPIO6: track 19.1 -> 17.0 mm
- net Net-(R3-Pad2): track 5.32 -> 7.31 mm
Other:
- board text added: "${REFERENCE}"

Commit message: actu
Parts:
- moved D1 3.52 mm to (187.6, 85.7)
Routing:
- net Net-(D1-K): track 48.1 -> 50.6 mm
- net Net-(D1-A): track 5.40 -> 7.62 mm
- net +5V: track 126.4 -> 128.0 mm
Changed lines of the file:
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@@
 	(footprint "LED_THT:LED_D3.0mm_Clear"
 		(layer "F.Cu")
-		(at 187.5 82.15 90)
+		(at 187.55 85.67 90)
 		(descr "LED, diameter 3.0mm, 2 pins, clear, generated by kicad-footprint-generator")
 		(tags "LED")
@@
 	)
 	(segment
-		(start 187.5 82.15)
-		(end 192.825 82.15)
-		(width 1)
-		(layer "B.Cu")
-		(net 1)
-	)
-	(segment
-		(start 192.825 82.15)
-		(end 194.7875 80.1875)
-		(width 1)
-		(layer "B.Cu")
-		(net 1)
-	)
-	(segment
 		(start 214.25 70.1)
 		(end 214.25 62.190999)
@@
 	)
 	(segment
+		(start 191.13 85.67)
+		(end 194.7875 82.0125)
+		(width 1)
+		(layer "B.Cu")
+		(net 1)
+	)
+	(segment
 		(start 194.7875 69.7)
 		(end 197.95 69.7)
@@
 	)
 	(segment
-		(start 194.7875 69.7)
-		(end 194.7875 80.1875)
+		(start 187.55 85.67)
+		(end 191.13 85.67)
+		(width 1)
+		(layer "B.Cu")
+		(net 1)
+	)
+	(segment
+		(start 194.7875 82.0125)
+		(end 194.7875 69.7)
 		(width 1)
 		(layer "B.Cu")
@@
 	)
 	(segment
-		(start 187.5025 79.6125)
-		(end 187.5 79.61)
+		(start 190.77 83.13)
+		(end 187.55 83.13)
 		(width 1)
 		(layer "B.Cu")
@@
 	)
 	(segment
+		(start 192.9 81)
+		(end 190.77 83.13)
+		(width 1)
+		(layer "B.Cu")
+		(net 2)
+	)
+	(segment
 		(start 192.9 79.6125)
-		(end 187.5025 79.6125)
+		(end 192.9 81)
 		(width 1)
 		(layer "B.Cu")
@@
 	)
 	(segment
-		(start 179.24 57.63)
-		(end 179.24 58.74)
+		(start 214.25 82.1)
+		(end 217.01 82.1)
 		(width 1)
 		(layer "B.Cu")
@@
 	)
 	(segment
+		(start 179.24 57.21)
+		(end 179.24 58.74)
+		(width 1)
+		(layer "B.Cu")
+		(net 3)
+	)
+	(segment
+		(start 214.9 56.18)
+		(end 180.27 56.18)
+		(width 1)
+		(layer "B.Cu")
+		(net 3)
+	)
+	(segment
+		(start 217.01 82.1)
+		(end 219.04 80.07)
+		(width 1)
+		(layer "B.Cu")
+		(net 3)
+	)
+	(segment
+		(start 219.04 80.07)
+		(end 219.04 60.32)
+		(width 1)
+		(layer "B.Cu")
+		(net 3)
+	)
+	(segment
 		(start 219.04 60.32)
 		(end 214.9 56.18)
@@
 	)
 	(segment
-		(start 214.25 82.1)
-		(end 217.01 82.1)
-		(width 1)
-		(layer "B.Cu")
-		(net 3)
-	)
-	(segment
-		(start 192.9125 69.7)
-		(end 192.9125 67.7275)
-		(width 0.75)
-		(layer "B.Cu")
-		(net 3)
-	)
-	(segment
 		(start 192.9125 69.7)
 		(end 192.9125 77.775)
@@
 	)
 	(segment
-		(start 202.0375 63.0325)
-		(end 202.0375 62.085)
+		(start 192.9125 66.1375)
+		(end 194.1 64.95)
 		(width 0.75)
-		(layer "B.Cu")
-		(net 3)
-	)
-	(segment
-		(start 180.69 56.18)
-		(end 179.24 57.63)
-		(width 1)
-		(layer "B.Cu")
-		(net 3)
-	)
-	(segment
-		(start 217.01 82.1)
-		(end 219.04 80.07)
-		(width 1)
 		(layer "B.Cu")
 		(net 3)
@@
 	)
 	(segment
+		(start 192.9125 69.7)
+		(end 192.9125 66.1375)
+		(width 0.75)
+		(layer "B.Cu")
+		(net 3)
+	)
+	(segment
 		(start 202.0375 62.085)
 		(end 200.895 62.085)
@@
 	)
 	(segment
-		(start 192.9125 67.7275)
-		(end 196.73 63.91)
-		(width 0.75)
-		(layer "B.Cu")
-		(net 3)
-	)
-	(segment
-		(start 196.73 63.91)
-		(end 201.16 63.91)
-		(width 0.75)
-		(layer "B.Cu")
-		(net 3)
-	)
-	(segment
-		(start 219.04 80.07)
-		(end 219.04 60.32)
-		(width 1)
-		(layer "B.Cu")
-		(net 3)
-	)
-	(segment
 		(start 214.81 87.66)
 		(end 214.81 92.95)
@@
 	)
 	(segment
-		(start 214.9 56.18)
-		(end 180.69 56.18)
+		(start 200.75 64.95)
+		(end 202.0375 63.6625)
+		(width 0.75)
+		(layer "B.Cu")
+		(net 3)
+	)
+	(segment
+		(start 180.27 56.18)
+		(end 179.24 57.21)
 		(width 1)
 		(layer "B.Cu")
@@
 	)
 	(segment
-		(start 201.16 63.91)
-		(end 202.0375 63.0325)
+		(start 194.1 64.95)
+		(end 200.75 64.95)
 		(width 0.75)
 		(layer "B.Cu")
+		(net 3)
+	)
+	(segment
+		(start 202.0375 63.6625)
+		(end 202.0375 62.085)
+		(width 0.75)
+		(layer "B.Cu")

Commit message: actu
Parts:
- removed U1: ESP8266-DEVKITC-02U-F, esp32:ESP8266NA
- added U2: ~, ESP32_Footprints:ESP32_30pin, F.Cu at (163.6, 71.3)
Routing:
- net GPIO6: track 17.0 -> 8.11 mm
- net +5V: track 128.0 -> 125.0 mm
- removed copper zone on B.Cu, net GND
Other:
- board size 70 x 45 mm -> 78.6 x 55.1 mm

Commit message: actu pcb
Parts:
- removed J3: Screw_Terminal_01x02, TerminalBlock:TerminalBlock_MaiXu_MX126-5.0-02P_1x02_P5.00mm
- added D2: LED IR, LED_THT:LED_D3.0mm_Clear, F.Cu at (180.9, 95.2)
- added Q1: BC337, Package_TO_SOT_THT:TO-92_Inline, F.Cu at (183.2, 75.2)
- added R4: 220, Resistor_SMD:R_0805_2012Metric, B.Cu at (178.3, 73.1)
- added R5: 47, Resistor_SMD:R_0805_2012Metric, B.Cu at (183.4, 82.8)
- moved D3 6.74 mm to (187.7, 72.5)
- moved R1 6.14 mm to (186.8, 78.9)
- moved Q2 5.34 mm to (209.8, 65.1)
- moved J1 5.08 mm to (209.7, 93.0)
- moved J2 5.08 mm to (192.4, 93.0)
- moved U5 5.08 mm to (193.8, 61.5)
- moved K1 4.48 mm to (211.8, 76.0)
- moved R2 3.67 mm to (204.9, 63.9)
- moved D1 1.73 mm to (189.3, 85.6), turned to 180 degrees
- moved U2 1.31 mm to (162.2, 71.3)
- moved R3 0.55 mm to (186.9, 62.1)
Connections:
- U2 pad 8: unconnected-(U2-GPIO25-Pad8) -> GPIO7
Routing:
- net Net-(D2-K): track 0.00 -> 21.5 mm
- net Net-(D2-A): track 0.00 -> 11.5 mm
- net GPIO6: track 8.11 -> 16.8 mm
- net Net-(D1-K): track 50.6 -> 43.7 mm
- net Net-(Q1-B): track 0.00 -> 4.90 mm
- net Net-(R3-Pad2): track 7.31 -> 2.77 mm
- net Net-(R2-Pad1): track 3.88 -> 8.28 mm
- net GPIO7: track 0.00 -> 4.16 mm
- net Net-(Q2-B): track 6.52 -> 4.06 mm
- net Net-(D1-A): track 7.62 -> 5.78 mm
- net +5V: track 125.0 -> 123.3 mm
- net COM: track 22.1 -> 22.7 mm
- net NO: track 14.1 -> 14.7 mm
- added copper zone on B.Cu, net GND
Other:
- board size 78.6 x 55.1 mm -> 73.6 x 55.1 mm

Commit message: act placa
Parts:
- moved R3 11.2 mm to (178.6, 69.5)
- moved U5 2.13 mm to (193.8, 63.6)
- moved D3 1.81 mm to (187.7, 74.3)
Routing:
- net GPIO6: track 16.8 -> 3.52 mm
- net Net-(R3-Pad2): track 2.77 -> 13.3 mm
- net +5V: track 123.3 -> 121.2 mm
- net Net-(D1-K): track 43.7 -> 42.5 mm
- net Net-(R2-Pad1): track 8.28 -> 7.34 mm
Other:
- board text added: "Rele-Wifi"
