File: Hardware/Rele wifi/Rele wifi 2/Rele wifi 2.kicad_pcb (KiCad board)
At the start: 2 copper layers, 70 x 50 mm, 15 parts, among them J1 Screw_Terminal_01x02, J2 Screw_Terminal_01x03, J3 Screw_Terminal_01x02, K1 G5LE-1, Q2 BC337, U1 ESP8266-DEVKITC-02U-F, U5 PC817

Commit message: actu 15/9
Parts:
- U1: value ESP8266-DEVKITC-02U-F -> ~; footprint ESP8266:ESP12F-Devkit-V3 -> ESP32_Footprints:ESP32_30pin
- moved C2 4.83 mm to (163.8, 53.3)
- moved R1 3.48 mm to (155.5, 46.4)
- moved R2 3.45 mm to (160.7, 42.0)
- moved D1 3.44 mm to (157.1, 41.8)
- moved C1 3.44 mm to (154.6, 54.3)
- moved R3 2.98 mm to (176.7, 46.3)
- moved U5 1.76 mm to (167.2, 47.7)
- moved U1 0.87 mm to (178.1, 71.4)
Connections:
- C1 pad 1: +5V -> VIN
- C2 pad 1: +5V -> VIN
- D3 pad 1: +5V -> VIN
- J1 pad 1: +5V -> VIN
- K1 pad 5: +5V -> VIN
- R1 pad 2: +5V -> VIN
- U1 pad 1: (no net) -> VIN
- U1 pad 10: (no net) -> unconnected-(U1-GPIO32-Pad10)
- U1 pad 11: (no net) -> unconnected-(U1-GPIO35-Pad11)
- U1 pad 12: (no net) -> unconnected-(U1-GPIO34-Pad12)
- U1 pad 13: (no net) -> unconnected-(U1-GPIO39-Pad13)
- U1 pad 14: (no net) -> unconnected-(U1-GPIO36-Pad14)
- U1 pad 15: (no net) -> unconnected-(U1-EN-Pad15)
- U1 pad 16: (no net) -> unconnected-(U1-3.3v-Pad16)
- U1 pad 17: (no net) -> unconnected-(U1-GND-Pad17)
- U1 pad 18: (no net) -> unconnected-(U1-GPIO15-Pad18)
- U1 pad 19: (no net) -> unconnected-(U1-GPIO2-Pad19)
- U1 pad 2: (no net) -> GND
- U1 pad 20: (no net) -> unconnected-(U1-GPIO4-Pad20)
- U1 pad 21: (no net) -> unconnected-(U1-GPIO16-Pad21)
- U1 pad 22: (no net) -> unconnected-(U1-GPIO17-Pad22)
- U1 pad 23: (no net) -> unconnected-(U1-GPIO5-Pad23)
- U1 pad 24: (no net) -> unconnected-(U1-GPIO18-Pad24)
- U1 pad 25: (no net) -> unconnected-(U1-GPIO19-Pad25)
- U1 pad 26: (no net) -> unconnected-(U1-GPIO21-Pad26)
- U1 pad 27: (no net) -> unconnected-(U1-GPIO3-Pad27)
- U1 pad 28: (no net) -> unconnected-(U1-GPIO1-Pad28)
- U1 pad 29: (no net) -> unconnected-(U1-GPIO22-Pad29)
- U1 pad 3: (no net) -> unconnected-(U1-GPIO13-Pad3)
- U1 pad 30: (no net) -> unconnected-(U1-GPIO23-Pad30)
- U1 pad 4: (no net) -> unconnected-(U1-GPIO12-Pad4)
- U1 pad 5: (no net) -> unconnected-(U1-GPIO14-Pad5)
- U1 pad 6: (no net) -> unconnected-(U1-GPIO27-Pad6)
- U1 pad 7: (no net) -> GPIO6
- U1 pad 8: (no net) -> unconnected-(U1-GPIO25-Pad8)
- U1 pad 9: (no net) -> unconnected-(U1-GPIO33-Pad9)
- U5 pad 4: +5V -> VIN
Routing:
- net VIN: track 0.00 -> 139.6 mm
- net +5V: track 129.3 -> 0.00 mm
- net GPIO6: track 0.00 -> 20.2 mm, vias 0 -> 2
- net Net-(Q2-B): track 3.10 -> 6.56 mm
- net Net-(D1-K): track 47.3 -> 50.7 mm
- net Net-(R2-Pad1): track 10.9 -> 13.7 mm
- net Net-(R3-Pad2): track 5.11 -> 3.90 mm
- net Net-(D1-A): track 18.7 -> 17.5 mm

Commit message: act placa
Parts:
- removed J3: Screw_Terminal_01x02, TerminalBlock:TerminalBlock_MaiXu_MX126-5.0-02P_1x02_P5.00mm
- added D2: LED, LED_THT:LED_D3.0mm_Clear, F.Cu at (217.2, 82.6)
- added J4: Conn_01x03_Pin, Connector_PinHeader_2.00mm:PinHeader_1x03_P2.00mm_Vertical, F.Cu at (217.2, 73.3)
- added R5: 220, Resistor_SMD:R_0805_2012Metric, B.Cu at (210.3, 82.7)
- added SW1: SW_Push, Button_Switch_THT:SW_PUSH_1P1T_6x3.5mm_H5.0_APEM_MJTP1250, F.Cu at (206.7, 73.3)
- moved J1 14.6 mm to (215.0, 65.6)
Connections:
- U1 pad 21: unconnected-(U1-GPIO16-Pad21) -> GPIO12
- U1 pad 22: unconnected-(U1-GPIO17-Pad22) -> GPIO14
- U1 pad 28: unconnected-(U1-GPIO1-Pad28) -> GPIO4
Routing:
- net GPIO14: track 0.00 -> 46.3 mm
- net GPIO12: track 0.00 -> 40.6 mm
- net GPIO4: track 0.00 -> 23.7 mm
- net VIN: track 139.6 -> 134.2 mm
- net Net-(D2-A): track 0.00 -> 3.49 mm
