File: Hardware/Rele wifi/Rele wifi sacha/Rele wifi 2.kicad_pcb (KiCad board)
At the start: 2 copper layers, 65 x 50 mm, 16 parts, among them J1 Screw_Terminal_01x02, J2 Screw_Terminal_01x03, J4 Conn_01x03_Pin, K1 G5LE-1, Q2 BC337, SW1 SW_Push, U5 PC817

Commit message: actu pcb
Parts:
- moved D1 1.84 mm to (210.2, 53.3)
- moved U5 0.95 mm to (204.3, 45.8)
- moved J2 0.60 mm to (158.3, 41.2)
- moved K1 0.60 mm to (187.5, 46.3)
- moved U1 0.54 mm to (178.6, 70.4)
- moved R1 0.44 mm to (212.9, 48.0)
- moved R3 0.43 mm to (195.8, 47.1)
- moved R4 0.31 mm to (198.4, 51.0)
- moved R2 0.28 mm to (206.0, 50.8)
- moved Q2 0.27 mm to (202.6, 52.9)
Routing:
- net GND: track 29.8 -> 31.8 mm
- net +5V: track 146.0 -> 147.5 mm
- net Net-(D1-A): track 5.42 -> 4.07 mm
- net Net-(R3-Pad2): track 3.81 -> 2.90 mm
- net Net-(R2-Pad1): track 8.24 -> 7.60 mm
- net Net-(Q2-B): track 2.89 -> 3.40 mm

Commit message: actu pcb
Parts:
- moved D2 2.70 mm to (207.9, 85.0), turned to 90 degrees
- moved R1 1.04 mm to (212.0, 47.6)
- moved R3 0.46 mm to (196.0, 46.7)
- moved U5 0.36 mm to (204.3, 45.4)
- moved R5 0.28 mm to (201.1, 79.4)
- moved SW1 0.18 mm to (207.6, 72.4)
Routing:
- net GND: track 31.8 -> 27.4 mm, vias 2 -> 0
- net GPIO14: track 48.8 -> 45.9 mm
- net Net-(D2-A): track 7.95 -> 7.10 mm
- net +5V: track 147.5 -> 146.6 mm
- net GPIO6: track 28.2 -> 28.8 mm

Commit message: actu
Routing:
- net +5V: track 146.6 -> 145.9 mm
Changed lines of the file:
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@@
+	)
+	(segment
+		(start 178.22 54.74)
+		(end 176.982277 55.977723)
+		(width 1)
+		(layer "B.Cu")
+		(net 9)
 	)
 	(segment
@@
 	)
 	(segment
+		(start 191.965 54.74)
+		(end 178.22 54.74)
+		(width 1)
+		(layer "B.Cu")
+		(net 9)
+	)
+	(segment
+		(start 192.03 54.675)
+		(end 191.965 54.74)
+		(width 1)
+		(layer "B.Cu")
+		(net 9)
+	)
+	(segment
 		(start 193.57 46.71)
 		(end 195.13 46.71)
@@
 	)
 	(segment
-		(start 191.965 54.74)
-		(end 178.22 54.74)
-		(width 1)
-		(layer "B.Cu")
-		(net 9)
-	)
-	(segment
 		(start 192.79 47.49)
 		(end 192.18 48.1)
@@
 	)
 	(segment
-		(start 192.03 54.675)
-		(end 191.965 54.74)
+		(start 192.04 48.24)
+		(end 192.04 51.21)
 		(width 1)
 		(layer "B.Cu")
@@
 	)
 	(segment
-		(start 178.22 54.74)
-		(end 176.982277 55.977723)
-		(width 1)
-		(layer "B.Cu")
-		(net 9)
-	)
-	(segment
-		(start 192.04 48.24)
-		(end 192.04 51.21)
-		(width 1)
-		(layer "B.Cu")
-		(net 9)
-	)
-	(segment
 		(start 196.955 46.71)
 		(end 199.5525 46.71)
@@
 	)
 	(segment
+		(start 214.23 64.35)
+		(end 214.23 47.74)
+		(width 1)
+		(layer "B.Cu")
+		(net 12)
+	)
+	(segment
 		(start 175.3 54.8)
 		(end 162.9 54.8)
@@
 	)
 	(segment
+		(start 213.1575 46.6675)
+		(end 211.98 46.6675)
+		(width 1)
+		(layer "B.Cu")
+		(net 12)
+	)
+	(segment
 		(start 214.45 77.02)
 		(end 211.3725 73.9425)
@@
 	)
 	(segment
-		(start 214.59 64.42)
-		(end 214.59 47.71)
+		(start 214.23 47.74)
+		(end 213.1575 46.6675)
 		(width 1)
 		(layer "B.Cu")
@@
 	)
 	(segment
-		(start 213.525 65.485)
-		(end 214.59 64.42)
+		(start 213.095 65.485)
+		(end 214.23 64.35)
 		(width 1)
 		(layer "B.Cu")
@@
 	(segment
 		(start 211.3725 65.485)
-		(end 213.525 65.485)
+		(end 213.095 65.485)
 		(width 1)
 		(layer "B.Cu")
@@
 	)
 	(segment
-		(start 213.5475 46.6675)
-		(end 211.98 46.6675)
-		(width 1)
-		(layer "B.Cu")
-		(net 12)
-	)
-	(segment
 		(start 161.642277 62.852277)
 		(end 164.275 65.485)
@@
 	)
 	(segment
-		(start 214.59 47.71)
-		(end 213.5475 46.6675)
-		(width 1)
-		(layer "B.Cu")
-		(net 12)
-	)
-	(segment
 		(start 207.88 82.43)
 		(end 206.22 82.43)
@@
 	)
 	(segment
+		(start 211.86 83.52)
+		(end 214.45 83.52)
+		(width 1)
+		(layer "B.Cu")
+		(net 37)
+	)
+	(segment
+		(start 180.03 77.29)
+		(end 205.63 77.29)
+		(width 1)
+		(layer "B.Cu")
+		(net 37)
+	)
+	(segment
 		(start 176.87 84.91)
 		(end 176.882277 84.897723)
@@
 	)
 	(segment
-		(start 206.18 77.29)
-		(end 212.41 83.52)
-		(width 1)
-		(layer "B.Cu")
-		(net 37)
-	)
-	(segment
-		(start 212.41 83.52)
-		(end 214.45 83.52)
+		(start 176.882277 84.897723)
+		(end 176.882277 80.437723)
 		(width 1)
 		(layer "B.Cu")
@@
 	)
 	(segment
-		(start 180.03 77.29)
-		(end 206.18 77.29)
-		(width 1)
-		(layer "B.Cu")
-		(net 37)
-	)
-	(segment
-		(start 176.882277 84.897723)
-		(end 176.882277 80.437723)
-		(width 1)
-		(layer "B.Cu")
+		(start 205.63 77.29)
+		(end 211.86 83.52)
+		(width 1)
+		(layer "B.Cu")

Commit message: actu pcb
Parts:
- moved J2 0.15 mm to (158.3, 41.0)
- moved K1 0.15 mm to (187.5, 46.1)
Routing:
- net GPIO6: track 28.8 -> 28.2 mm

Commit message: actu pcb
Routing:
- net GPIO6: track 28.2 -> 27.3 mm
Changed lines of the file:
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@@
+			)
+		)
+		(fp_text user "GND"
+			(at 10.02754 14.780187 270)
+			(unlocked yes)
+			(layer "F.SilkS")
+			(effects
+				(font
+					(size 1 1.1)
+					(thickness 0.1)
+				)
+				(justify left bottom)
 			)
 		)
@@
 		(fp_text user "GND"
 			(at -11.9 14.680187 270)
-			(unlocked yes)
-			(layer "F.SilkS")
-			(effects
-				(font
-					(size 1 1.1)
-					(thickness 0.1)
-				)
-				(justify left bottom)
-			)
-		)
-		(fp_text user "GND"
-			(at 10.02754 14.780187 270)
 			(unlocked yes)
 			(layer "F.SilkS")
@@
 	)
 	(segment
-		(start 208.9575 44.12)
-		(end 208.9675 44.13)
-		(width 1)
-		(layer "B.Cu")
-		(net 8)
-	)
-	(segment
 		(start 205.98 49.8675)
 		(end 205.98 45.56)
@@
 	)
 	(segment
-		(start 192.18 48.1)
-		(end 192.04 48.24)
-		(width 1)
-		(layer "B.Cu")
-		(net 9)
-	)
-	(segment
-		(start 192.18 48.1)
-		(end 193.57 46.71)
-		(width 1)
-		(layer "B.Cu")
-		(net 9)
-	)
-	(segment
 		(start 191.965 54.74)
 		(end 178.22 54.74)
@@
 	)
 	(segment
+		(start 192.04 48.24)
+		(end 193.57 46.71)
+		(width 1)
+		(layer "B.Cu")
+		(net 9)
+	)
+	(segment
 		(start 192.03 54.675)
 		(end 191.965 54.74)
@@
 	)
 	(segment
-		(start 192.79 47.49)
-		(end 192.18 48.1)
-		(width 1)
-		(layer "B.Cu")
-		(net 9)
-	)
-	(segment
 		(start 177.089813 55.870187)
 		(end 178.22 54.74)
@@
 	)
 	(segment
-		(start 214.23 64.35)
-		(end 214.23 47.74)
+		(start 213.1575 46.6675)
+		(end 211.98 46.6675)
+		(width 1)
+		(layer "B.Cu")
+		(net 12)
+	)
+	(segment
+		(start 210.48 40.6)
+		(end 194.9175 40.6)
 		(width 1)
 		(layer "B.Cu")
@@
 	)
 	(segment
+		(start 214.69 64.49)
+		(end 214.69 48.2)
+		(width 1)
+		(layer "B.Cu")
+		(net 12)
+	)
+	(segment
 		(start 164.275 65.485)
 		(end 211.3725 65.485)
@@
 	)
 	(segment
-		(start 213.1575 46.6675)
-		(end 211.98 46.6675)
-		(width 1)
-		(layer "B.Cu")
-		(net 12)
-	)
-	(segment
 		(start 161.849813 63.059813)
 		(end 164.275 65.485)
@@
 	)
 	(segment
-		(start 214.23 47.74)
-		(end 213.1575 46.6675)
+		(start 213.695 65.485)
+		(end 214.69 64.49)
 		(width 1)
 		(layer "B.Cu")
@@
 	)
 	(segment
+		(start 211.98 42.1)
+		(end 210.48 40.6)
+		(width 1)
+		(layer "B.Cu")
+		(net 12)
+	)
+	(segment
 		(start 161.849813 55.850187)
 		(end 162.9 54.8)
@@
 	)
 	(segment
+		(start 211.3725 65.485)
+		(end 213.695 65.485)
+		(width 1)
+		(layer "B.Cu")
+		(net 12)
+	)
+	(segment
 		(start 211.98 46.6675)
-		(end 211.98 41.5)
-		(width 1)
-		(layer "B.Cu")
-		(net 12)
-	)
-	(segment
-		(start 213.095 65.485)
-		(end 214.23 64.35)
-		(width 1)
-		(layer "B.Cu")
-		(net 12)
-	)
-	(segment
-		(start 211.08 40.6)
-		(end 194.9175 40.6)
+		(end 211.98 42.1)
 		(width 1)
 		(layer "B.Cu")
@@
 	)
 	(segment
-		(start 211.98 41.5)
-		(end 211.08 40.6)
+		(start 214.69 48.2)
+		(end 213.1575 46.6675)
 		(width 1)
 		(layer "B.Cu")
@@
 		(start 175.3 54.8)
 		(end 177.99 52.11)
-		(width 1)
-		(layer "B.Cu")
-		(net 12)
-	)
-	(segment
-		(start 211.3725 65.485)
-		(end 213.095 65.485)
 		(width 1)
 		(layer "B.Cu")
@@
 		(polygon
 			(pts
-				(xy 152.35 36.936077) (xy 191.53 37.03) (xy 191.27 55.97) (xy 152.34 56)
-			)
-		)
+				(xy 152.35 36.936077) (xy 191.69 37.06) (xy 191.52 56.01) (xy 152.34 56)
+			)
+		)

Commit message: actu pcb
Parts:
- moved R5 2.29 mm to (198.8, 79.4)
- moved R4 0.95 mm to (198.4, 50.0)
- moved D1 0.72 mm to (209.5, 53.3)
- moved R2 0.36 mm to (206.3, 50.8)
Routing:
- net GPIO4: track 12.1 -> 9.77 mm
- net Net-(D2-A): track 7.10 -> 9.40 mm
- net Net-(D1-A): track 3.66 -> 4.33 mm
Changed lines of the file:
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@@
 	(footprint "LED_THT:LED_D3.0mm_Clear"
 		(layer "F.Cu")
-		(at 210.18 53.27 90)
+		(at 209.46 53.26 90)
 		(descr "LED, diameter 3.0mm, 2 pins, clear, generated by kicad-footprint-generator")
 		(tags "LED")
@@
 	(footprint "Resistor_SMD:R_0805_2012Metric"
 		(layer "B.Cu")
-		(at 201.1225 79.39 180)
+		(at 198.83 79.39 180)
 		(descr "Resistor SMD 0805 (2012 Metric), square (rectangular) end terminal, IPC-7351 nominal, (Body size source: IPC-SM-782 page 72, https://www.pcb-3d.com/wordpress/wp-content/uploads/ipc-sm-782a_amendment_1_and_2.pdf), generated with kicad-footprint-generator")
 		(tags "resistor")
@@
 	(footprint "Resistor_SMD:R_0805_2012Metric"
 		(layer "B.Cu")
-		(at 205.98 50.78 -90)
+		(at 206.34 50.78 -90)
 		(descr "Resistor SMD 0805 (2012 Metric), square (rectangular) end terminal, IPC_7351 nominal, (Body size source: IPC-SM-782 page 72, https://www.pcb-3d.com/wordpress/wp-content/uploads/ipc-sm-782a_amendment_1_and_2.pdf), generated with kicad-footprint-generator")
 		(tags "resistor")
@@
 	(footprint "Resistor_SMD:R_0805_2012Metric"
 		(layer "B.Cu")
-		(at 198.37 50.96)
+		(at 198.41 50.01)
 		(descr "Resistor SMD 0805 (2012 Metric), square (rectangular) end terminal, IPC_7351 nominal, (Body size source: IPC-SM-782 page 72, https://www.pcb-3d.com/wordpress/wp-content/uploads/ipc-sm-782a_amendment_1_and_2.pdf), generated with kicad-footprint-generator")
 		(tags "resistor")
@@
 	)
 	(segment
-		(start 210.18 49.14)
-		(end 210.8275 48.4925)
+		(start 210.1675 48.4925)
+		(end 211.98 48.4925)
 		(width 1)
 		(layer "B.Cu")
@@
 	)
 	(segment
-		(start 210.18 50.73)
-		(end 210.18 49.14)
+		(start 209.46 50.72)
+		(end 209.46 49.2)
 		(width 1)
 		(layer "B.Cu")
@@
 	)
 	(segment
-		(start 210.8275 48.4925)
-		(end 211.98 48.4925)
+		(start 209.46 49.2)
+		(end 210.1675 48.4925)
 		(width 1)
 		(layer "B.Cu")
@@
 	)
 	(segment
-		(start 191.3675 53.3)
-		(end 190.36 52.2925)
+		(start 194.9175 53.3)
+		(end 191.81 53.3)
 		(width 1)
 		(layer "B.Cu")
@@
 	)
 	(segment
-		(start 194.9875 53.23)
-		(end 194.9175 53.3)
+		(start 190.36 42.08)
+		(end 188.39 40.11)
+		(width 1)
+		(layer "B.Cu")
+		(net 2)
+	)
+	(segment
+		(start 191.81 53.3)
+		(end 190.36 51.85)
+		(width 1)
+		(layer "B.Cu")
+		(net 2)
+	)
+	(segment
+		(start 190.36 51.85)
+		(end 190.36 42.08)
 		(width 1)
 		(layer "B.Cu")
@@
 	)
 	(segment
-		(start 190.36 52.2925)
-		(end 190.36 42.84)
+		(start 194.9875 53.23)
+		(end 194.9175 53.3)
 		(width 1)
 		(layer "B.Cu")
@@
 	)
 	(segment
-		(start 210.18 53.27)
-		(end 202.63 53.27)
+		(start 209.46 53.26)
+		(end 202.62 53.26)
 		(width 1)
 		(layer "B.Cu")
@@
 	)
 	(segment
-		(start 194.9175 53.3)
-		(end 191.3675 53.3)
-		(width 1)
-		(layer "B.Cu")
-		(net 2)
-	)
-	(segment
-		(start 190.36 42.84)
-		(end 187.63 40.11)
+		(start 202.62 53.26)
+		(end 202.59 53.23)
 		(width 1)
 		(layer "B.Cu")
@@
 	)
 	(segment
-		(start 187.63 40.11)
+		(start 188.39 40.11)
 		(end 185.47 40.11)
 		(width 1)
@@
 	)
 	(segment
-		(start 205.98 51.6925)
+		(start 206.34 51.6925)
 		(end 202.6225 51.6925)
 		(width 1)
@@
 	)
 	(segment
-		(start 205.98 49.8675)
-		(end 205.98 45.56)
+		(start 206.34 45.2)
+		(end 207.42 44.12)
 		(width 1)
 		(layer "B.Cu")
@@
 	)
 	(segment
-		(start 207.42 44.12)
-		(end 208.9575 44.12)
+		(start 206.34 49.8675)
+		(end 206.34 45.2)
 		(width 1)
 		(layer "B.Cu")
@@
 	)
 	(segment
-		(start 205.98 45.56)
-		(end 207.42 44.12)
+		(start 207.42 44.12)
+		(end 208.9575 44.12)
 		(width 1)
 		(layer "B.Cu")
@@
 	)
 	(segment
-		(start 199.2825 50.96)
-		(end 200.37 50.96)
+		(start 199.3225 50.01)
+		(end 202.57 50.01)
 		(width 1)
 		(layer "B.Cu")
@@
 	)
 	(segment
-		(start 202.58 50.02)
-		(end 202.59 50.03)
-		(width 1)
-		(layer "B.Cu")
-		(net 11)
-	)
-	(segment
-		(start 200.37 50.96)
-		(end 201.3 50.03)
-		(width 1)
-		(layer "B.Cu")
-		(net 11)
-	)
-	(segment
-		(start 201.3 50.03)
+		(start 202.57 50.01)
 		(end 202.59 50.03)
 		(width 1)
@@
 	)
 	(segment
-		(start 207.88 82.43)
-		(end 206.22 82.43)
+		(start 206.22 82.43)
+		(end 203.18 79.39)
 		(width 1)
 		(layer "B.Cu")
@@
 	)
 	(segment
-		(start 206.22 82.43)
-		(end 203.18 79.39)
+		(start 203.18 79.39)
+		(end 199.7425 79.39)
 		(width 1)
 		(layer "B.Cu")
@@
 	)
 	(segment
-		(start 203.18 79.39)
-		(end 202.035 79.39)
+		(start 207.88 82.43)
+		(end 206.22 82.43)
 		(width 1)
 		(layer "B.Cu")
@@
 	(segment
 		(start 194.7075 79.39)
-		(end 200.21 79.39)
+		(end 197.9175 79.39)
 		(width 1)
 		(layer "B.Cu")
