File: Hardware/Rele wifi/Rele wifi sacha/Rele wifi 2.kicad_pcb (KiCad board)
At the start: 2 copper layers, 65 x 50 mm, 16 parts, among them J1 Screw_Terminal_01x02, J2 Screw_Terminal_01x03, J4 Conn_01x03_Pin, K1 G5LE-1, Q2 BC337, SW1 SW_Push, U5 PC817

Commit message: actu pcb
Parts:
- moved R2 2.63 mm to (206.3, 48.1)
- moved R3 1.11 mm to (196.0, 44.6)
- moved U5 1.09 mm to (204.2, 43.4)
- moved R1 1.07 mm to (211.9, 45.6)
- moved R4 0.87 mm to (198.8, 49.1)
- moved D3 0.84 mm to (194.9, 39.8)
- moved Q2 0.78 mm to (202.6, 52.1)
- moved D1 0.77 mm to (211.9, 52.5)
- moved SW1 0.35 mm to (207.9, 71.5)
Routing:
- net GPIO14: track 45.6 -> 50.5 mm
- net GPIO12: track 42.0 -> 44.4 mm
- net Net-(R2-Pad1): track 8.66 -> 6.96 mm
- net Net-(Q2-B): track 3.74 -> 5.17 mm
- net GPIO6: track 28.5 -> 29.4 mm
- net Net-(D1-K): track 37.4 -> 36.7 mm

Commit message: actu pcb 5/10
Parts:
- moved D1 20.3 mm to (196.1, 39.8), turned to -90 degrees
- moved Q2 16.0 mm to (213.2, 40.2), turned to -90 degrees
- moved R1 15.8 mm to (196.1, 45.8), turned to -90 degrees
- moved R4 15.8 mm to (214.1, 45.6), turned to 180 degrees
- moved D3 13.2 mm to (191.3, 52.4), turned to 90 degrees
- moved R3 12.1 mm to (205.8, 51.8)
- moved R5 9.53 mm to (208.1, 83.5)
- moved J4 6.99 mm to (213.5, 71.0), turned to -90 degrees
- moved R2 6.67 mm to (205.5, 41.5), turned to 0 degrees
- moved SW1 5.46 mm to (208.0, 76.9)
- moved D2 5.02 mm to (214.5, 83.5)
- moved U5 4.71 mm to (205.2, 48.0), turned to 180 degrees
- moved K1 1.79 mm to (185.7, 46.1)
- moved J1 1.09 mm to (211.4, 64.6)
- moved J2 0.25 mm to (158.0, 41.0)
Connections:
- U1 pad 21: GPIO12 -> GPIO14
- U1 pad 22: GPIO14 -> GPIO12
Routing:
- net +5V: track 144.7 -> 111.0 mm, vias 0 -> 2
- net GPIO4: track 10.4 -> 19.9 mm
- net GPIO6: track 29.4 -> 36.7 mm, vias 2 -> 0
- net Net-(D1-K): track 36.7 -> 29.7 mm
- net GPIO12: track 44.4 -> 37.4 mm
- net Net-(D2-A): track 9.59 -> 2.96 mm
- net GPIO14: track 50.5 -> 45.5 mm
- net Net-(R3-Pad2): track 2.60 -> 7.41 mm
- net Net-(R2-Pad1): track 6.96 -> 11.1 mm
- net Net-(Q2-B): track 5.17 -> 6.78 mm
- net NO: track 15.4 -> 13.8 mm
- net NC: track 15.4 -> 13.8 mm
- net COM: track 29.2 -> 27.7 mm
- net Net-(D1-A): track 3.45 -> 2.53 mm

Commit message: act sacha
Parts:
- moved R1 5.03 mm to (191.3, 44.2)
- moved R3 1.86 mm to (205.0, 50.1)
- moved U5 1.62 mm to (204.7, 46.4)
- moved SW1 1.07 mm to (208.1, 78.0)
- moved J4 1.01 mm to (213.6, 72.0)
- moved D2 0.78 mm to (215.2, 83.9)
- moved R5 0.66 mm to (208.6, 83.9)
- moved R2 0.51 mm to (205.0, 41.5)
- moved J1 0.41 mm to (211.8, 64.6)
- moved U1 0.35 mm to (178.8, 70.1)
- moved J2 0.18 mm to (157.9, 40.8)
- moved K1 0.18 mm to (185.6, 45.9)
Routing:
- net +5V: track 111.0 -> 116.6 mm
- net Net-(D1-A): track 2.53 -> 5.26 mm
- net Net-(R2-Pad1): track 11.1 -> 9.08 mm
- net GPIO4: track 19.9 -> 18.2 mm
- net GPIO6: track 36.7 -> 37.7 mm
- net GPIO14: track 45.5 -> 44.8 mm
- net GPIO12: track 37.4 -> 36.8 mm
- net Net-(Q2-B): track 6.78 -> 7.32 mm

Commit message: actu 6/10
Parts:
- moved Q2 6.03 mm to (207.2, 40.2)
- moved J1 5.92 mm to (211.7, 58.6)
- moved J4 5.18 mm to (214.6, 66.9), turned to 0 degrees
- moved R4 4.77 mm to (210.7, 42.3), turned to -90 degrees
- moved U5 3.98 mm to (200.8, 47.2)
- moved R2 3.49 mm to (201.5, 41.5)
- moved R3 3.10 mm to (202.2, 51.6), turned to 90 degrees
- moved R1 0.82 mm to (191.3, 45.1)
Routing:
- net GPIO14: track 44.8 -> 50.9 mm
- net Net-(D1-K): track 29.7 -> 24.5 mm
- net GPIO6: track 37.7 -> 32.9 mm
- net +5V: track 116.6 -> 113.8 mm
- net Net-(Q2-B): track 7.32 -> 4.83 mm
- net Net-(Q2-E): track 2.41 -> 3.50 mm
- net Net-(D1-A): track 5.26 -> 6.04 mm
- net Net-(R2-Pad1): track 9.08 -> 9.80 mm
