File: Hardware/Rele wifi/Rele wifi sacha/Rele wifi 2.kicad_sch (KiCad schematic)
At the start: 18 parts, among them J1 Screw_Terminal_01x02, J2 Screw_Terminal_01x03, J4 Conn_01x03_Pin, K1 G5LE-1, Q2 BC337, SW1 SW_Push, U5 PC817

Commit message: actu
Parts:
- removed C1: 100nF, Capacitor_THT:C_Disc_D4.7mm_W2.5mm_P5.00mm, symbol Device:C
- removed C2: 10uF, Capacitor_THT:CP_Radial_D5.0mm_P2.00mm, symbol Device:C_Polarized
Connections:
- net GND: now also U1.17 (GND)
Changed lines of the file:
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@@
-	)
-	(junction
-		(at 93.98 24.13)
-		(diameter 0)
-		(color 0 0 0 0)
 	)
 	(junction
@@
 	)
 	(junction
-		(at 80.01 24.13)
-		(diameter 0)
-		(color 0 0 0 0)
-	)
-	(junction
 		(at 102.87 46.99)
 		(diameter 0)
@@
 		(color 0 0 0 0)
 	)
-	(junction
-		(at 87.63 36.83)
-		(diameter 0)
-		(color 0 0 0 0)
-	)
 	(wire
 		(pts
@@
 	(wire
 		(pts
-			(xy 93.98 36.83) (xy 87.63 36.83)
-		)
-		(stroke
-			(width 0)
-			(type default)
-		)
-	)
-	(wire
-		(pts
-			(xy 80.01 24.13) (xy 87.63 24.13)
-		)
-		(stroke
-			(width 0)
-			(type default)
-		)
-	)
-	(wire
-		(pts
 			(xy 165.1 33.02) (xy 168.91 33.02)
 		)
@@
 	(wire
 		(pts
-			(xy 93.98 24.13) (xy 102.87 24.13)
+			(xy 87.63 24.13) (xy 102.87 24.13)
 		)
 		(stroke
@@
 	(wire
 		(pts
-			(xy 93.98 24.13) (xy 93.98 26.67)
-		)
-		(stroke
-			(width 0)
-			(type default)
-		)
-	)
-	(wire
-		(pts
-			(xy 93.98 34.29) (xy 93.98 36.83)
-		)
-		(stroke
-			(width 0)
-			(type default)
-		)
-	)
-	(wire
-		(pts
-			(xy 80.01 36.83) (xy 87.63 36.83)
-		)
-		(stroke
-			(width 0)
-			(type default)
-		)
-	)
-	(wire
-		(pts
 			(xy 259.08 59.69) (xy 260.35 59.69)
 		)
@@
 	(wire
 		(pts
-			(xy 76.2 24.13) (xy 80.01 24.13)
+			(xy 76.2 24.13) (xy 87.63 24.13)
 		)
 		(stroke
@@
 	(wire
 		(pts
-			(xy 87.63 24.13) (xy 93.98 24.13)
-		)
-		(stroke
-			(width 0)
-			(type default)
-		)
-	)
-	(wire
-		(pts
-			(xy 80.01 24.13) (xy 80.01 26.67)
-		)
-		(stroke
-			(width 0)
-			(type default)
-		)
-	)
-	(wire
-		(pts
 			(xy 91.44 54.61) (xy 95.25 54.61)
 		)
@@
 	(wire
 		(pts
-			(xy 87.63 38.1) (xy 87.63 36.83)
-		)
-		(stroke
-			(width 0)
-			(type default)
-		)
-	)
-	(wire
-		(pts
-			(xy 80.01 34.29) (xy 80.01 36.83)
+			(xy 87.63 35.56) (xy 87.63 38.1)
 		)
 		(stroke
@@
 	(wire
 		(pts
-			(xy 87.63 35.56) (xy 87.63 36.83)
-		)
-		(stroke
-			(width 0)
-			(type default)
-		)
-	)
-	(wire
-		(pts
 			(xy 168.91 30.48) (xy 171.45 30.48)
 		)
@@
 		(property "Intersheetrefs" "${INTERSHEET_REFS}"
 			(at 265.9357 38.1 0)
+			(effects
+				(font
+					(size 1.27 1.27)
+				)
+				(justify left)
+				(hide yes)
+			)
+		)
+	)
+	(global_label "GND"
+		(shape input)
+		(at 231.14 59.69 0)
+		(fields_autoplaced yes)
+		(effects
+			(font
+				(size 1.27 1.27)
+			)
+			(justify left)
+		)
+		(property "Intersheetrefs" "${INTERSHEET_REFS}"
+			(at 237.9957 59.69 0)
 			(effects
 				(font
@@
 	)
 	(symbol
-		(lib_id "Device:C_Polarized")
-		(at 80.01 30.48 0)
-		(unit 1)
-		(exclude_from_sim no)
-		(in_bom yes)
-		(on_board yes)
-		(dnp no)
-		(property "Reference" "C2"
-			(at 83.058 25.146 0)
-			(effects
-				(font
-					(size 1.27 1.27)
-				)
-				(justify left)
-			)
-		)
-		(property "Value" "10uF"
-			(at 81.788 27.5591 0)
-			(effects
-				(font
-					(size 1.27 1.27)
-				)
-				(justify left)
-			)
-		)
-		(property "Footprint" "Capacitor_THT:CP_Radial_D5.0mm_P2.00mm"
-			(at 80.9752 34.29 0)
-			(effects
-				(font
-					(size 1.27 1.27)
-				)
-				(hide yes)
-			)
-		)
-		(property "Datasheet" "~"
-			(at 80.01 30.48 0)
-			(effects
-				(font
-					(size 1.27 1.27)
-				)
-				(hide yes)
-			)
-		)
-		(property "Description" "Polarized capacitor"
-			(at 80.01 30.48 0)
-			(effects
-				(font
-					(size 1.27 1.27)
-				)
-				(hide yes)
-			)
-		)
-		(pin "1"
-		)
-		(pin "2"
-		)
-		(instances
-			(project ""
-				(path "/1a5734b3-aec8-47c8-9ec1-200a88fc117c"
-					(reference "C2")
-					(unit 1)
-				)
-			)
-		)
-	)
-	(symbol
 		(lib_id "power:+5V")
 		(at 168.91 33.02 180)
@@
 					(unit 1)
 				)
-			)
-		)
-	)
-	(symbol
-		(lib_id "Device:C")
-		(at 93.98 30.48 0)
-		(unit 1)
-		(exclude_from_sim no)
-		(in_bom yes)
-		(on_board yes)
-		(dnp no)
-		(property "Reference" "C1"
-			(at 97.79 29.21 0)
-			(effects
-				(font
-					(size 1.27 1.27)
-				)
-				(justify left)
-			)
-		)
-		(property "Value" "100nF"
-			(at 95.758 34.544 0)
-			(effects
-				(font
-					(size 1.27 1.27)
-				)
-				(justify left)
-			)
-		)
-		(property "Footprint" "Capacitor_THT:C_Disc_D4.7mm_W2.5mm_P5.00mm"
-			(at 94.9452 34.29 0)
-			(effects
-				(font
-					(size 1.27 1.27)
-				)
-				(hide yes)
-			)
-		)
-		(property "Datasheet" "~"
-			(at 93.98 30.48 0)
-			(effects
-				(font
-					(size 1.27 1.27)
-				)
-				(hide yes)
-			)
-		)
-		(property "Description" "Unpolarized capacitor"
-			(at 93.98 30.48 0)
-			(effects
-				(font
-					(size 1.27 1.27)
-				)
-				(hide yes)
-			)
-		)
-		(pin "2"
-		)
-		(pin "1"
-		)
-		(instances
-			(project ""
-				(path "/1a5734b3-aec8-47c8-9ec1-200a88fc117c"
-					(reference "C1")
-					(unit 1)
-				)

Commit message: actu pcb
Parts:
- J1: footprint TerminalBlock:TerminalBlock_MaiXu_MX126-5.0-02P_1x02_P5.00mm -> TerminalBlock_Phoenix:TerminalBlock_Phoenix_MKDS-1,5-2-5.08_1x02_P5.08mm_Horizontal
- J2: footprint TerminalBlock:TerminalBlock_MaiXu_MX126-5.0-03P_1x03_P5.00mm -> TerminalBlock_Phoenix:TerminalBlock_Phoenix_MKDS-1,5-3-5.08_1x03_P5.08mm_Horizontal
- J4: footprint Connector_PinHeader_2.00mm:PinHeader_1x03_P2.00mm_Vertical -> Connector_PinSocket_2.54mm:PinSocket_1x03_P2.54mm_Vertical

Commit message: actu pcb
Connections:
- net NC: now also J2.1 (Pin_1); no longer J2.3 (Pin_3)
- net NO: now also J2.3 (Pin_3); no longer J2.1 (Pin_1)
Changed lines of the file:
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@@
 	(global_label "NO"
 		(shape input)
-		(at 264.16 21.59 180)
+		(at 264.16 26.67 180)
 		(fields_autoplaced yes)
 		(effects
@@
 		)
 		(property "Intersheetrefs" "${INTERSHEET_REFS}"
-			(at 258.5138 21.59 0)
+			(at 258.5138 26.67 0)
 			(effects
 				(font
@@
 	(global_label "NC"
 		(shape input)
-		(at 264.16 26.67 180)
+		(at 264.16 21.59 180)
 		(fields_autoplaced yes)
 		(effects
@@
 		)
 		(property "Intersheetrefs" "${INTERSHEET_REFS}"
-			(at 258.5743 26.67 0)
+			(at 258.5743 21.59 0)
 			(effects
 				(font

Commit message: actu pcb 5/10
Connections:
- net GPIO12: now also U1.22 (GPIO17); no longer U1.21 (GPIO16)
- net GPIO14: now also U1.21 (GPIO16); no longer U1.22 (GPIO17)
Changed lines of the file:
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@@
 	(global_label "GPIO14"
 		(shape input)
-		(at 231.14 46.99 0)
+		(at 231.14 49.53 0)
 		(fields_autoplaced yes)
 		(effects
@@
 		)
 		(property "Intersheetrefs" "${INTERSHEET_REFS}"
-			(at 241.0195 46.99 0)
+			(at 241.0195 49.53 0)
 			(effects
 				(font
@@
 	(global_label "GPIO12"
 		(shape input)
-		(at 231.14 49.53 0)
+		(at 231.14 46.99 0)
 		(fields_autoplaced yes)
 		(effects
@@
 		)
 		(property "Intersheetrefs" "${INTERSHEET_REFS}"
-			(at 241.0195 49.53 0)
+			(at 241.0195 46.99 0)
 			(effects
 				(font
