File: Hardware/Rele wifi/Rele Wifi/Rele wifi.kicad_sch (KiCad schematic)
At the start: 15 parts, among them J1 Screw_Terminal_01x02, J2 Screw_Terminal_01x03, K1 G5LE-1, Q1 BC337, Q2 BC337, U5 PC817

Commit message: act placa
Connections:
- net COM: now also J2.2 (Pin_2); no longer J2.3 (Pin_3)
- net NC: now also J2.3 (Pin_3); no longer J2.2 (Pin_2)
Changed lines of the file:
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@@
 	(global_label "NC"
 		(shape input)
-		(at 234.95 30.48 180)
+		(at 234.95 33.02 180)
 		(fields_autoplaced yes)
 		(effects
@@
 		)
 		(property "Intersheetrefs" "${INTERSHEET_REFS}"
-			(at 229.3643 30.48 0)
+			(at 229.3643 33.02 0)
 			(effects
 				(font
@@
 	(global_label "COM"
 		(shape input)
-		(at 234.95 33.02 180)
+		(at 234.95 30.48 180)
 		(fields_autoplaced yes)
 		(effects
@@
 		)
 		(property "Intersheetrefs" "${INTERSHEET_REFS}"
-			(at 227.9129 33.02 0)
+			(at 227.9129 30.48 0)
 			(effects
 				(font

Commit message: actu nachin
Parts:
- added J3: Conn_01x02_Pin, Connector_PinHeader_2.54mm:PinHeader_1x02_P2.54mm_Vertical, symbol Connector:Conn_01x02_Pin
- U5: footprint Package_SO:SOP-4_4.4x2.6mm_P1.27mm -> Package_DIP:DIP-4_W7.62mm_SMDSocket_SmallPads
Connections:
- net GND: now also U2.17 (GND), J3.2 (Pin_2)
- net GPIO6: now also U2.22 (GPIO17); no longer U2.7 (GPIO26)
- net GPIO7: now also U2.21 (GPIO16); no longer U2.8 (GPIO25)
- net at U2.15 (EN): now also J3.1 (Pin_1)
Changed lines of the file:
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@@
+	(wire
+		(pts
+			(xy 35.56 30.48) (xy 40.64 30.48)
+		)
+		(stroke
+			(width 0)
+			(type default)
+		)
+	)
 	(wire
 		(pts
@@
 	(global_label "GPIO6"
 		(shape input)
-		(at 40.64 50.8 180)
+		(at 68.58 50.8 0)
 		(fields_autoplaced yes)
 		(effects
@@
 				(size 1.27 1.27)
 			)
-			(justify right)
+			(justify left)
 		)
 		(property "Intersheetrefs" "${INTERSHEET_REFS}"
-			(at 31.97 50.8 0)
-			(effects
-				(font
-					(size 1.27 1.27)
-				)
-				(justify right)
+			(at 77.25 50.8 0)
+			(effects
+				(font
+					(size 1.27 1.27)
+				)
+				(justify left)
 				(hide yes)
 			)
@@
 	(global_label "GPIO7"
 		(shape input)
-		(at 40.64 48.26 180)
+		(at 68.58 53.34 0)
 		(fields_autoplaced yes)
 		(effects
@@
 				(size 1.27 1.27)
 			)
-			(justify right)
+			(justify left)
 		)
 		(property "Intersheetrefs" "${INTERSHEET_REFS}"
-			(at 31.97 48.26 0)
-			(effects
-				(font
-					(size 1.27 1.27)
-				)
-				(justify right)
+			(at 77.25 53.34 0)
+			(effects
+				(font
+					(size 1.27 1.27)
+				)
+				(justify left)
 				(hide yes)
 			)
@@
 			)
 		)
-		(property "Footprint" "Package_SO:SOP-4_4.4x2.6mm_P1.27mm"
+		(property "Footprint" "Package_DIP:DIP-4_W7.62mm_SMDSocket_SmallPads"
 			(at 120.65 60.96 0)
 			(effects
@@
 				(path "/ffdbb2c2-c0c7-4e42-be77-90fd93012b1e"
 					(reference "#PWR01")
+					(unit 1)
+				)
+			)
+		)
+	)
+	(symbol
+		(lib_id "power:GND")
+		(at 35.56 33.02 0)
+		(unit 1)
+		(exclude_from_sim no)
+		(in_bom yes)
+		(on_board yes)
+		(dnp no)
+		(fields_autoplaced yes)
+		(property "Reference" "#PWR07"
+			(at 35.56 39.37 0)
+			(effects
+				(font
+					(size 1.27 1.27)
+				)
+				(hide yes)
+			)
+		)
+		(property "Value" "GND"
+			(at 35.56 38.1 0)
+			(effects
+				(font
+					(size 1.27 1.27)
+				)
+			)
+		)
+		(property "Footprint" ""
+			(at 35.56 33.02 0)
+			(effects
+				(font
+					(size 1.27 1.27)
+				)
+				(hide yes)
+			)
+		)
+		(property "Datasheet" ""
+			(at 35.56 33.02 0)
+			(effects
+				(font
+					(size 1.27 1.27)
+				)
+				(hide yes)
+			)
+		)
+		(property "Description" "Power symbol creates a global label with name \"GND\" , ground"
+			(at 35.56 33.02 0)
+			(effects
+				(font
+					(size 1.27 1.27)
+				)
+				(hide yes)
+			)
+		)
+		(pin "1"
+		)
+		(instances
+			(project "Rele wifi"
+				(path "/ffdbb2c2-c0c7-4e42-be77-90fd93012b1e"
+					(reference "#PWR07")
+					(unit 1)
+				)
+			)
+		)
+	)
+	(symbol
+		(lib_id "power:GND")
+		(at 68.58 63.5 90)
+		(unit 1)
+		(exclude_from_sim no)
+		(in_bom yes)
+		(on_board yes)
+		(dnp no)
+		(fields_autoplaced yes)
+		(property "Reference" "#PWR06"
+			(at 74.93 63.5 0)
+			(effects
+				(font
+					(size 1.27 1.27)
+				)
+				(hide yes)
+			)
+		)
+		(property "Value" "GND"
+			(at 72.39 63.4999 90)
+			(effects
+				(font
+					(size 1.27 1.27)
+				)
+				(justify right)
+			)
+		)
+		(property "Footprint" ""
+			(at 68.58 63.5 0)
+			(effects
+				(font
+					(size 1.27 1.27)
+				)
+				(hide yes)
+			)
+		)
+		(property "Datasheet" ""
+			(at 68.58 63.5 0)
+			(effects
+				(font
+					(size 1.27 1.27)
+				)
+				(hide yes)
+			)
+		)
+		(property "Description" "Power symbol creates a global label with name \"GND\" , ground"
+			(at 68.58 63.5 0)
+			(effects
+				(font
+					(size 1.27 1.27)
+				)
+				(hide yes)
+			)
+		)
+		(pin "1"
+		)
+		(instances
+			(project "Rele wifi"
+				(path "/ffdbb2c2-c0c7-4e42-be77-90fd93012b1e"
+					(reference "#PWR06")
 					(unit 1)
 				)
@@
 					(unit 1)
 				)
+			)
+		)
+	)
+	(symbol
+		(lib_id "Connector:Conn_01x02_Pin")
+		(at 30.48 30.48 0)
+		(unit 1)
+		(exclude_from_sim no)
+		(in_bom yes)
+		(on_board yes)
+		(dnp no)
+		(fields_autoplaced yes)
+		(property "Reference" "J3"
+			(at 31.115 25.4 0)
+			(effects
+				(font
+					(size 1.27 1.27)
+				)
+			)
+		)
+		(property "Value" "Conn_01x02_Pin"
+			(at 31.115 27.94 0)
+			(effects
+				(font
+					(size 1.27 1.27)
+				)
+			)
+		)
+		(property "Footprint" "Connector_PinHeader_2.54mm:PinHeader_1x02_P2.54mm_Vertical"
+			(at 30.48 30.48 0)
+			(effects
+				(font
+					(size 1.27 1.27)
+				)
+				(hide yes)
+			)
+		)
+		(property "Datasheet" "~"
+			(at 30.48 30.48 0)
+			(effects
+				(font
+					(size 1.27 1.27)
+				)
+				(hide yes)
+			)
+		)
+		(property "Description" "Generic connector, single row, 01x02, script generated"
+			(at 30.48 30.48 0)
+			(effects
+				(font
+					(size 1.27 1.27)
+				)
+				(hide yes)
+			)
+		)
+		(pin "2"
+		)
+		(pin "1"
+		)
+		(instances
+			(project ""
+				(path "/ffdbb2c2-c0c7-4e42-be77-90fd93012b1e"
+					(reference "J3")
+					(unit 1)
+				)

Commit message: actu nachin
Parts:
- U5: footprint Package_DIP:DIP-4_W7.62mm_SMDSocket_SmallPads -> Package_SO:SOP-4_7.5x4.1mm_P2.54mm
Changed lines of the file:
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@@
 			)
 		)
-		(property "Footprint" "Package_DIP:DIP-4_W7.62mm_SMDSocket_SmallPads"
+		(property "Footprint" "Package_SO:SOP-4_7.5x4.1mm_P2.54mm"
 			(at 120.65 60.96 0)
 			(effects

Commit message: actu
Parts:
- D3: footprint Diode_SMD:D_0805_2012Metric -> Diode_THT:D_DO-41_SOD81_P12.70mm_Horizontal
Connections:
- net GPIO6 renamed GPIO12
- net GPIO12: now also U2.21 (GPIO16); no longer U2.22 (GPIO17)
- net GPIO7 renamed GPIO13
- net GPIO13: now also U2.22 (GPIO17); no longer U2.21 (GPIO16)
Other:
- moved on the sheet: D3
Changed lines of the file:
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@@
 	(wire
 		(pts
-			(xy 156.21 30.48) (xy 156.21 40.64)
+			(xy 156.21 30.48) (xy 156.21 36.83)
 		)
 		(stroke
@@
 	(wire
 		(pts
-			(xy 156.21 48.26) (xy 156.21 50.8)
+			(xy 156.21 44.45) (xy 156.21 50.8)
 		)
 		(stroke
@@
 		)
 	)
-	(global_label "GPIO6"
+	(global_label "GPIO12"
 		(shape input)
 		(at 107.95 53.34 180)
@@
 		)
 		(property "Intersheetrefs" "${INTERSHEET_REFS}"
-			(at 99.28 53.34 0)
+			(at 98.0705 53.34 0)
 			(effects
 				(font
@@
 		)
 	)
-	(global_label "GPIO7"
+	(global_label "GPIO13"
 		(shape input)
 		(at 220.98 96.52 180)
@@
 		)
 		(property "Intersheetrefs" "${INTERSHEET_REFS}"
-			(at 212.31 96.52 0)
+			(at 211.1005 96.52 0)
 			(effects
 				(font
@@
 		)
 	)
-	(global_label "GPIO6"
+	(global_label "GPIO12"
 		(shape input)
-		(at 68.58 50.8 0)
+		(at 68.58 53.34 0)
 		(fields_autoplaced yes)
 		(effects
@@
 		)
 		(property "Intersheetrefs" "${INTERSHEET_REFS}"
-			(at 77.25 50.8 0)
+			(at 78.4595 53.34 0)
 			(effects
 				(font
@@
 		)
 	)
-	(global_label "GPIO7"
+	(global_label "GPIO13"
 		(shape input)
-		(at 68.58 53.34 0)
+		(at 68.58 50.8 0)
 		(fields_autoplaced yes)
 		(effects
@@
 		)
 		(property "Intersheetrefs" "${INTERSHEET_REFS}"
-			(at 77.25 53.34 0)
+			(at 78.4595 50.8 0)
 			(effects
 				(font
@@
 		(lib_name "1N4007_1")
 		(lib_id "local_lib:1N4007")
-		(at 156.21 44.45 270)
+		(at 156.21 40.64 270)
 		(unit 1)
 		(exclude_from_sim no)
@@
 		(fields_autoplaced yes)
 		(property "Reference" "D3"
-			(at 158.75 43.815 90)
+			(at 158.75 40.005 90)
 			(effects
 				(font
@@
 		)
 		(property "Value" "1N4007"
-			(at 158.75 46.355 90)
+			(at 158.75 42.545 90)
 			(effects
 				(font
@@
 			)
 		)
-		(property "Footprint" "Diode_SMD:D_0805_2012Metric"
-			(at 151.765 44.45 0)
+		(property "Footprint" "Diode_THT:D_DO-41_SOD81_P12.70mm_Horizontal"
+			(at 151.765 40.64 0)
 			(effects
 				(font
@@
 		)
 		(property "Datasheet" "http://www.vishay.com/docs/88503/1n4001.pdf"
-			(at 156.21 44.45 0)
+			(at 156.21 40.64 0)
 			(effects
 				(font
@@
 		)
 		(property "Description" ""
-			(at 156.21 44.45 0)
+			(at 156.21 40.64 0)
 			(effects
 				(font
@@
 		)
 		(property "Sim.Device" "D"
-			(at 156.21 44.45 0)
+			(at 156.21 40.64 0)
 			(effects
 				(font
@@
 		)
 		(property "Sim.Pins" "1=K 2=A"
-			(at 156.21 44.45 0)
-			(effects
-				(font
+			(at 156.21 40.64 0)
+			(effects
+				(font
