File: Hardware/Rele wifi/Rele Wifi/Rele wifi.kicad_pcb (KiCad board)
At the start: 2 copper layers, 73.6 x 55.1 mm, 15 parts, among them J1 Screw_Terminal_01x02, J2 Screw_Terminal_01x03, K1 G5LE-1, Q1 BC337, Q2 BC337, U5 PC817

Commit message: actu
Parts:
- moved J1 43.1 mm to (213.0, 50.0), turned to 180 degrees
- moved J2 10.4 mm to (201.9, 97.3)
- moved K1 3.80 mm to (208.1, 75.2), turned to 0 degrees
Routing:
- net +5V: track 120.9 -> 62.2 mm
- net NC: track 25.2 -> 0.00 mm
- net COM: track 22.7 -> 0.00 mm
- net NO: track 13.0 -> 0.00 mm

Commit message: act placa
Parts:
- moved D1 9.63 mm to (189.3, 95.2)
- moved J2 9.36 mm to (210.7, 94.1), turned to 180 degrees
- moved K1 8.85 mm to (205.7, 66.7)
- moved Q2 6.89 mm to (205.8, 59.6)
- moved R2 6.89 mm to (200.8, 58.4)
- moved U5 5.61 mm to (193.1, 59.0)
- moved J1 5.06 mm to (207.9, 50.0)
- moved R3 0.87 mm to (178.4, 68.6), turned to 90 degrees
Connections:
- J2 pad 2: NC -> COM
- J2 pad 3: COM -> NC
Routing:
- net +5V: track 62.2 -> 102.8 mm
- net COM: track 0.00 -> 27.4 mm
- net NO: track 0.00 -> 13.6 mm
- net NC: track 0.00 -> 13.6 mm
- net Net-(D1-A): track 5.78 -> 15.4 mm
- net Net-(D1-K): track 43.2 -> 50.8 mm
- net Net-(R3-Pad2): track 12.0 -> 17.7 mm
- net Net-(R2-Pad1): track 7.93 -> 3.64 mm
- net GPIO6: track 3.52 -> 4.31 mm

Commit message: actu nachin
Parts:
- added J3: Conn_01x02_Pin, Connector_PinHeader_2.54mm:PinHeader_1x02_P2.54mm_Vertical, F.Cu at (179.2, 96.1)
- U5: footprint Package_SO:SOP-4_4.4x2.6mm_P1.27mm -> Package_DIP:DIP-4_W7.62mm_SMDSocket_SmallPads
- moved R3 5.81 mm to (184.2, 68.6)
- moved D3 4.43 mm to (192.0, 75.6)
- moved R1 4.43 mm to (191.0, 80.1)
- moved R5 4.43 mm to (187.7, 84.1)
- moved D1 4.27 mm to (193.5, 95.7)
- moved D2 4.27 mm to (185.1, 95.7)
- moved R4 3.44 mm to (181.2, 74.9), turned to -90 degrees
- moved U2 2.70 mm to (159.7, 72.2), turned to 0 degrees
- moved J2 2.17 mm to (212.8, 94.1)
- moved K1 2.17 mm to (207.8, 66.7)
- moved Q1 1.98 mm to (185.2, 75.2)
- moved U5 0.71 mm to (193.1, 59.7)
Connections:
- U2 pad 15: unconnected-(U2-EN-Pad15) -> Net-(J3-Pin_1)
- U2 pad 17: unconnected-(U2-GND-Pad17) -> GND
- U2 pad 21: unconnected-(U2-GPIO16-Pad21) -> GPIO7
- U2 pad 22: unconnected-(U2-GPIO17-Pad22) -> GPIO6
- U2 pad 7: GPIO6 -> unconnected-(U2-GPIO26-Pad7)
- U2 pad 8: GPIO7 -> unconnected-(U2-GPIO25-Pad8)
Routing:
- net Net-(J3-Pin_1): track 0.00 -> 67.6 mm, vias 0 -> 2
- net +5V: track 102.8 -> 164.7 mm
- net GND: track 0.00 -> 31.6 mm, vias 0 -> 2
- net Net-(R3-Pad2): track 17.7 -> 10.6 mm
- net GPIO6: track 4.31 -> 11.1 mm
- net Net-(D1-K): track 50.8 -> 46.3 mm
- net GPIO7: track 4.16 -> 6.57 mm
- net Net-(D2-K): track 21.7 -> 20.3 mm
- net Net-(Q1-B): track 4.90 -> 3.99 mm
- net Net-(D2-A): track 11.5 -> 10.7 mm
- net Net-(D1-A): track 15.4 -> 14.7 mm
- net Net-(R2-Pad1): track 3.64 -> 3.02 mm

Commit message: actu nachin
Parts:
- U5: footprint Package_DIP:DIP-4_W7.62mm_SMDSocket_SmallPads -> Package_SO:SOP-4_7.5x4.1mm_P2.54mm
- moved U5 0.99 mm to (192.1, 59.7)
Routing:
- net Net-(R3-Pad2): track 10.6 -> 9.03 mm

Commit message: actu
Parts:
- D3: footprint Diode_SMD:D_0805_2012Metric -> Diode_THT:D_DO-41_SOD81_P12.70mm_Horizontal; moved to F.Cu
- moved D3 16.6 mm to (200.8, 61.6)
- moved Q2 7.81 mm to (213.5, 58.3)
- moved R2 6.72 mm to (207.5, 59.0)
- moved R4 4.85 mm to (181.2, 70.0), turned to 90 degrees
- moved U2 3.99 mm to (163.5, 71.1), turned to 180 degrees
- moved R3 2.93 mm to (184.2, 65.7)
- moved J1 0.69 mm to (208.3, 49.5)
- moved U5 0.55 mm to (192.1, 60.2)
Connections:
- R3 pad 1: GPIO6 -> GPIO12
- R4 pad 2: GPIO7 -> GPIO13
- U2 pad 21: GPIO7 -> GPIO12
- U2 pad 22: GPIO6 -> GPIO13
Routing:
- net Net-(J3-Pin_1): track 67.6 -> 9.02 mm, vias 2 -> 0
- net +5V: track 164.6 -> 110.1 mm
- net GPIO12: track 0.00 -> 35.9 mm
- net GPIO13: track 0.00 -> 33.0 mm
- net GND: track 31.6 -> 5.25 mm
- net GPIO6: track 11.1 -> 0.00 mm
- net Net-(D1-K): track 46.3 -> 53.9 mm
- net Net-(R2-Pad1): track 3.13 -> 9.80 mm
- net GPIO7: track 6.57 -> 0.00 mm
- net Net-(R3-Pad2): track 9.03 -> 5.88 mm
- net Net-(Q1-B): track 3.99 -> 6.38 mm
- net Net-(Q2-B): track 4.06 -> 5.84 mm

Commit message: actu pcb
Routing:
- net +5V: track 110.1 -> 110.8 mm
- net Net-(D1-K): track 53.9 -> 54.5 mm
Changed lines of the file:
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@@
-	)
-	(segment
-		(start 206.55 61.56)
-		(end 213.46 61.56)
-		(width 1)
-		(layer "B.Cu")
-		(net 1)
 	)
 	(segment
@@
 	)
 	(segment
+		(start 201.85 68.69625)
+		(end 201.85 65.22)
+		(width 1)
+		(layer "B.Cu")
+		(net 1)
+	)
+	(segment
 		(start 192.9275 89.8475)
 		(end 193.52 90.44)
@@
 	)
 	(segment
-		(start 201.85 68.69625)
-		(end 201.85 66.26)
-		(width 1)
-		(layer "B.Cu")
-		(net 1)
-	)
-	(segment
 		(start 192.9275 72.8525)
 		(end 194.14 71.64)
@@
 	)
 	(segment
+		(start 205.51 61.56)
+		(end 213.46 61.56)
+		(width 1)
+		(layer "B.Cu")
+		(net 1)
+	)
+	(segment
 		(start 192.9275 75.6)
 		(end 192.9275 89.8475)
@@
 	)
 	(segment
-		(start 201.85 66.26)
-		(end 206.55 61.56)
+		(start 201.85 65.22)
+		(end 205.51 61.56)
 		(width 1)
 		(layer "B.Cu")
@@
 	)
 	(segment
+		(start 194.72 69.59)
+		(end 196.79 67.52)
+		(width 1)
+		(layer "B.Cu")
+		(net 3)
+	)
+	(segment
+		(start 200.68 61.51)
+		(end 200.78 61.61)
+		(width 1)
+		(layer "B.Cu")
+		(net 3)
+	)
+	(segment
+		(start 193.41 54.090187)
+		(end 193.41 55.080561)
+		(width 1)
+		(layer "B.Cu")
+		(net 3)
+	)
+	(segment
+		(start 189.5125 79.2175)
+		(end 191.01 79.2175)
+		(width 1)
+		(layer "B.Cu")
+		(net 3)
+	)
+	(segment
+		(start 213.92 49.46)
+		(end 217.13 52.67)
+		(width 1)
+		(layer "B.Cu")
+		(net 3)
+	)
+	(segment
+		(start 196.7775 61.51)
+		(end 200.68 61.51)
+		(width 1)
+		(layer "B.Cu")
+		(net 3)
+	)
+	(segment
+		(start 175.46754 54.090187)
+		(end 192.1 54.090187)
+		(width 1)
+		(layer "B.Cu")
+		(net 3)
+	)
+	(segment
+		(start 206.809813 54.090187)
+		(end 208.33 52.57)
+		(width 1)
+		(layer "B.Cu")
+		(net 3)
+	)
+	(segment
+		(start 193.250187 60.170187)
+		(end 194.59 61.51)
+		(width 1)
+		(layer "B.Cu")
+		(net 3)
+	)
+	(segment
+		(start 217.13 67.57)
+		(end 216.00375 68.69625)
+		(width 1)
+		(layer "B.Cu")
+		(net 3)
+	)
+	(segment
+		(start 196.9075 61.64)
+		(end 196.7775 61.51)
+		(width 1)
+		(layer "B.Cu")
+		(net 3)
+	)
+	(segment
+		(start 191.01 79.2175)
+		(end 191.01 71.36)
+		(width 1)
+		(layer "B.Cu")
+		(net 3)
+	)
+	(segment
+		(start 193.41 55.080561)
+		(end 193.250187 55.240374)
+		(width 1)
+		(layer "B.Cu")
+		(net 3)
+	)
+	(segment
+		(start 192.1 54.090187)
+		(end 193.41 54.090187)
+		(width 1)
+		(layer "B.Cu")
+		(net 3)
+	)
+	(segment
+		(start 208.33 52.57)
+		(end 208.33 49.47)
+		(width 1)
+		(layer "B.Cu")
+		(net 3)
+	)
+	(segment
+		(start 217.13 52.67)
+		(end 217.13 67.57)
+		(width 1)
+		(layer "B.Cu")
+		(net 3)
+	)
+	(segment
+		(start 193.250187 55.43)
+		(end 193.250187 55.240374)
+		(width 1)
+		(layer "B.Cu")
+		(net 3)
+	)
+	(segment
+		(start 193.250187 55.240374)
+		(end 192.1 54.090187)
+		(width 1)
+		(layer "B.Cu")
+		(net 3)
+	)
+	(segment
+		(start 196.7775 67.5075)
+		(end 196.79 67.52)
+		(width 1)
+		(layer "B.Cu")
+		(net 3)
+	)
+	(segment
+		(start 187.66 81.07)
+		(end 189.5125 79.2175)
+		(width 1)
+		(layer "B.Cu")
+		(net 3)
+	)
+	(segment
+		(start 187.66 83.1675)
+		(end 187.66 81.07)
+		(width 1)
+		(layer "B.Cu")
+		(net 3)
+	)
+	(segment
+		(start 193.250187 55.43)
+		(end 193.250187 60.170187)
+		(width 1)
+		(layer "B.Cu")
+		(net 3)
+	)
+	(segment
 		(start 208.32 49.46)
 		(end 213.92 49.46)
@@
 	)
 	(segment
-		(start 194.72 69.59)
-		(end 196.79 67.52)
-		(width 1)
-		(layer "B.Cu")
-		(net 3)
-	)
-	(segment
-		(start 200.68 61.51)
-		(end 200.78 61.61)
-		(width 1)
-		(layer "B.Cu")
-		(net 3)
-	)
-	(segment
-		(start 193.41 54.090187)
-		(end 193.41 55.080561)
-		(width 1)
-		(layer "B.Cu")
-		(net 3)
-	)
-	(segment
-		(start 189.5125 79.2175)
-		(end 191.01 79.2175)
-		(width 1)
-		(layer "B.Cu")
-		(net 3)
-	)
-	(segment
-		(start 216.72 52.26)
-		(end 216.72 67.3)
-		(width 1)
-		(layer "B.Cu")
-		(net 3)
-	)
-	(segment
-		(start 196.7775 61.51)
-		(end 200.68 61.51)
-		(width 1)
-		(layer "B.Cu")
-		(net 3)
-	)
-	(segment
-		(start 216.72 67.3)
-		(end 215.32375 68.69625)
-		(width 1)
-		(layer "B.Cu")
-		(net 3)
-	)
-	(segment
-		(start 175.46754 54.090187)
-		(end 192.1 54.090187)
-		(width 1)
-		(layer "B.Cu")
-		(net 3)
-	)
-	(segment
-		(start 215.32375 68.69625)
+		(start 216.00375 68.69625)
 		(end 213.85 68.69625)
 		(width 1)
 		(layer "B.Cu")
-		(net 3)
-	)
-	(segment
-		(start 206.809813 54.090187)
-		(end 208.33 52.57)
-		(width 1)
-		(layer "B.Cu")
-		(net 3)
-	)
-	(segment
-		(start 193.250187 60.170187)
-		(end 194.59 61.51)
-		(width 1)
-		(layer "B.Cu")
-		(net 3)
-	)
-	(segment
-		(start 196.9075 61.64)
-		(end 196.7775 61.51)
-		(width 1)
-		(layer "B.Cu")
-		(net 3)
-	)
-	(segment
-		(start 191.01 79.2175)
-		(end 191.01 71.36)
-		(width 1)
-		(layer "B.Cu")
-		(net 3)
-	)
-	(segment
-		(start 193.41 55.080561)
-		(end 193.250187 55.240374)
-		(width 1)
-		(layer "B.Cu")
-		(net 3)
-	)
-	(segment
-		(start 192.1 54.090187)
-		(end 193.41 54.090187)
-		(width 1)
-		(layer "B.Cu")
-		(net 3)
-	)
-	(segment
-		(start 208.33 52.57)
-		(end 208.33 49.47)
-		(width 1)
-		(layer "B.Cu")
-		(net 3)
-	)
-	(segment
-		(start 193.250187 55.43)
-		(end 193.250187 55.240374)
-		(width 1)
-		(layer "B.Cu")
-		(net 3)
-	)
-	(segment
-		(start 213.92 49.46)
-		(end 216.72 52.26)
-		(width 1)
-		(layer "B.Cu")
-		(net 3)
-	)
-	(segment
-		(start 193.250187 55.240374)
-		(end 192.1 54.090187)
-		(width 1)
-		(layer "B.Cu")
-		(net 3)
-	)
-	(segment
-		(start 196.7775 67.5075)
-		(end 196.79 67.52)
-		(width 1)
-		(layer "B.Cu")
-		(net 3)
-	)
-	(segment
-		(start 187.66 81.07)
-		(end 189.5125 79.2175)
-		(width 1)
-		(layer "B.Cu")
-		(net 3)
-	)
-	(segment
-		(start 187.66 83.1675)
-		(end 187.66 81.07)
-		(width 1)
-		(layer "B.Cu")
-		(net 3)
-	)
-	(segment
-		(start 193.250187 55.43)
-		(end 193.250187 60.170187)
-		(width 1)
-		(layer "B.Cu")
